File: mic.kicad_pcb (KiCad board)
At the start: 2 copper layers, 38 parts, among them J2 USB_C_Receptacle_USB2.0_14P, SW1 SW_Push, U1 TS5A3159ADBVR, U2 INA826AID, U3 PCM2902CDBR, U4 TLV70033_SOT23-5, Y1 12MHz

Commit message: v1 board layout
Parts:
- added J1: AudioPlug3, Connector_Audio:Jack_3.5mm_QingPu_WQP-PJ398SM_Vertical_CircularHoles, F.Cu at (146.2, 83.0)
- J2: value USB_C_Receptacle_USB2.0_14P -> USB_C_Receptacle_USB2.0_16P
- moved R6 98.7 mm to (143.3, 105.4), turned to 90 degrees
- moved R5 98.3 mm to (147.0, 100.2), turned to -90 degrees
- moved R12 93.6 mm to (107.2, 83.5)
- moved R13 91.3 mm to (108.5, 79.5)
- moved U2 86.4 mm to (138.0, 102.1), turned to 0 degrees
- moved RV1 84.2 mm to (154.0, 85.0)
- moved C10 82.5 mm to (141.5, 64.2), turned to -90 degrees
- moved R4 82.1 mm to (137.5, 107.2)
- moved C9 64.8 mm to (126.3, 64.5), turned to -90 degrees
- moved C4 64.8 mm to (121.8, 64.0), turned to 90 degrees
- moved C5 56.4 mm to (127.8, 74.3), turned to 90 degrees
- moved C12 54.7 mm to (123.5, 74.5), turned to 90 degrees
- moved C8 49.4 mm to (141.2, 71.8), turned to 90 degrees
- moved C13 49.1 mm to (140.5, 74.2)
- moved C14 48.5 mm to (140.5, 78.5)
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Connections:
- J2 pad A8: (no net) -> unconnected-(J2-SBU1-PadA8)
- J2 pad B8: (no net) -> unconnected-(J2-SBU2-PadB8)
Routing:
- net Net-(R4-Pad1): track 3.52 -> 36.7 mm
- net Net-(J2-CC1): track 0.00 -> 26.4 mm
- net Net-(U3-VINL): track 0.00 -> 17.0 mm
- net Net-(U3-XTO): track 5.23 -> 19.3 mm
- net Earth: track 0.00 -> 14.0 mm
- net +5V: track 19.3 -> 32.6 mm
- net Net-(U3-VCCCI): track 0.00 -> 12.7 mm
- net Net-(C11-Pad1): track 0.00 -> 11.8 mm
- net Net-(U3-XTI): track 5.29 -> 14.2 mm
- net Net-(U3-VCCP1I): track 0.00 -> 8.43 mm
- net Net-(U2-RG_2): track 0.00 -> 8.16 mm
- net Net-(U3-VCCP2I): track 0.00 -> 7.01 mm
- net Net-(J2-D--PadA7): track 9.76 -> 14.7 mm, vias 0 -> 2
- net Net-(U3-VDDI): track 0.00 -> 4.88 mm
- net Net-(U2-+IN): track 0.00 -> 3.91 mm
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
Commit message: alt board version finished
Parts:
- removed the R4 at (137.5, 107.2)
- removed the R4 at (114.5, 89.2)
- added R4: 470R, Resistor_THT:R_Axial_DIN0204_L3.6mm_D1.6mm_P2.54mm_Vertical, F.Cu at (168.0, 81.0)
- RV1: footprint Potentiometer_THT:Potentiometer_ACP_CA9-V10_Vertical -> Potentiometer_THT:Potentiometer_Alps_RK097_Single_Horizontal
- SW1: footprint Button_Switch_THT:SW_DIP_SPSTx01_Piano_10.8x4.1mm_W7.62mm_P2.54mm -> Button_Switch_THT:SW_Tactile_SPST_Angled_PTS645Vx83-2LFS
- moved C3 64.3 mm to (175.8, 58.0), turned to 0 degrees
- moved C12 60.5 mm to (183.8, 80.2), turned to 0 degrees
- moved U4 58.8 mm to (169.8, 65.9), turned to 90 degrees
- moved R1 58.7 mm to (171.8, 59.8), turned to 180 degrees
- moved R11 55.9 mm to (178.2, 70.8), turned to -90 degrees
- moved U1 55.3 mm to (176.9, 63.3)
- moved C1 52.6 mm to (169.2, 62.2), turned to 0 degrees
- moved R3 50.6 mm to (178.3, 68.5), turned to 180 degrees
- moved MK2 48.8 mm to (168.0, 47.6), turned to -90 degrees
- moved C2 47.7 mm to (160.5, 63.2)
- moved R2 46.4 mm to (175.8, 66.2), turned to 0 degrees
- moved R8 46.0 mm to (151.8, 66.2)
- moved U2 46.0 mm to (173.2, 72.5), turned to 180 degrees
- moved R7 45.2 mm to (151.7, 64.0)
- moved R12 45.0 mm to (151.0, 73.0), turned to -90 degrees
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Routing:
- net Net-(U3-VOUTR): track 0.00 -> 72.8 mm
- net +5V: track 32.6 -> 103.2 mm, vias 0 -> 3
- net Net-(U3-VOUTL): track 0.00 -> 60.4 mm
- net Net-(R2-Pad1): track 8.09 -> 45.6 mm
- net Net-(D1-A): track 2.99 -> 35.0 mm
- net Net-(R4-Pad1): track 36.7 -> 6.76 mm
- net +3.3V: track 8.25 -> 31.8 mm, vias 0 -> 2
- net Net-(J2-CC1): track 26.4 -> 10.8 mm, vias 0 -> 1
- net Net-(U3-VCCXI): track 3.71 -> 17.9 mm
- net Net-(U3-VCOM): track 4.11 -> 15.8 mm
- net Net-(U2-REF): track 6.48 -> 17.4 mm
- net Net-(U2-VOUT): track 0.00 -> 9.19 mm
- net Net-(U3-VCCP1I): track 8.43 -> 15.4 mm
- net Net-(U3-VCCP2I): track 7.01 -> 12.6 mm
- net Net-(C1-Pad1): track 10.2 -> 4.84 mm
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- added copper zone on B.Cu, net Earth
- added copper zone on F.Cu, net Earth

Commit message: some fixes, will need help
Other:
- board outline added: 50 x 50 mm
Changed lines of the file:
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@@
 		)
 		(fill no)
-		(layer "F.Cu")
+		(layer "Edge.Cuts")
 	)
 	(segment

Commit message: some fixes
Parts:
- removed R9: 2k2, Resistor_THT:R_Axial_DIN0204_L3.6mm_D1.6mm_P2.54mm_Vertical
- added C15: 4u7, Capacitor_THT:C_Disc_D3.4mm_W2.1mm_P2.50mm, F.Cu at (168.2, 86.7)
- C4: value 1u -> 10u
- SW1: footprint Button_Switch_THT:SW_Tactile_SPST_Angled_PTS645Vx83-2LFS -> Button_Switch_THT:SW_Tactile_SPST_Angled_PTS645Vx58-2LFS
- moved C9 1.77 mm to (153.2, 87.0)
- moved R4 1.25 mm to (169.2, 81.0)
Connections:
- C9 pad 1: Net-(C9-Pad1) -> Net-(U3-VCOM)
Routing:
- net Net-(U3-VOUTR): track 72.8 -> 66.8 mm
- net Net-(U3-VOUTL): track 60.4 -> 54.5 mm
- net Net-(D1-A): track 35.0 -> 29.4 mm
- net +5V: track 103.2 -> 107.5 mm, vias 3 -> 2
- net Net-(U2-REF): track 17.4 -> 21.3 mm
- net Net-(C9-Pad1): track 2.77 -> 0.00 mm
- net Net-(U3-VCOM): track 15.8 -> 13.6 mm
- net +3.3V: track 31.8 -> 29.9 mm
- net Net-(U2-RG_2): track 12.2 -> 10.7 mm
- net Net-(R4-Pad1): track 6.76 -> 5.51 mm
- net Net-(C11-Pad1): track 7.59 -> 6.90 mm

Commit message: alt_1 V1
Parts:
- C11, C12: value 220u -> 470u; footprint Capacitor_THT:C_Disc_D3.4mm_W2.1mm_P2.50mm -> Capacitor_THT:CP_Radial_D8.0mm_P3.50mm
- moved C11 4.26 mm to (183.9, 58.8)
- moved C12 3.04 mm to (183.2, 83.2)
- turned C3 to 90 degrees
Routing:
- net Net-(C11-Pad1): track 6.90 -> 11.3 mm
- net Net-(C12-Pad2): track 2.88 -> 6.09 mm
- net Net-(U3-VOUTR): track 66.8 -> 69.9 mm
- net Net-(U3-VOUTL): track 54.5 -> 52.7 mm
