File: mic.kicad_sch (KiCad schematic)
At the start: 38 parts, among them J1 AudioPlug3, J2 USB_C_Receptacle_USB2.0_16P, SW1 SW_Push, U1 TS5A3159ADBVR, U2 INA826AID, U3 PCM2902CDBR, U4 TLV70033_SOT23-5, Y1 12MHz

Commit message: v1 board layout
Other:
- moved on the sheet: C4, C5, C6, C7, C8, J1

Commit message: alt board version finished
Parts:
- RV1: footprint Potentiometer_THT:Potentiometer_ACP_CA9-V10_Vertical -> Potentiometer_THT:Potentiometer_Alps_RK097_Single_Horizontal
- SW1: footprint Button_Switch_THT:SW_DIP_SPSTx01_Piano_10.8x4.1mm_W7.62mm_P2.54mm -> Button_Switch_THT:SW_Tactile_SPST_Angled_PTS645Vx58-2LFS
Changed lines of the file:
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@@
 			)
 		)
-		(property "Footprint" "Potentiometer_THT:Potentiometer_ACP_CA9-V10_Vertical"
+		(property "Footprint" "Potentiometer_THT:Potentiometer_Alps_RK097_Single_Horizontal"
 			(at 102.87 99.06 0)
 			(hide yes)
@@
 			)
 		)
-		(property "Footprint" "Button_Switch_THT:SW_DIP_SPSTx01_Piano_10.8x4.1mm_W7.62mm_P2.54mm"
+		(property "Footprint" "Button_Switch_THT:SW_Tactile_SPST_Angled_PTS645Vx58-2LFS"
 			(at 69.85 92.71 0)
 			(hide yes)

Commit message: some fixes
Parts:
- removed R9: 2k2, Resistor_THT:R_Axial_DIN0204_L3.6mm_D1.6mm_P2.54mm_Vertical, symbol Device:R
- added C15: 4u7, Capacitor_THT:C_Disc_D3.4mm_W2.1mm_P2.50mm, symbol Device:C
- C11, C12: value 220u -> 470u; footprint Capacitor_THT:C_Disc_D3.4mm_W2.1mm_P2.50mm -> Capacitor_THT:CP_Radial_D10.0mm_P5.00mm
- C4: value 1u -> 10u
Connections:
- net Earth: now also C15.1
- net at R5.2, R6.2, U2.6 (REF): now also C15.2
- net at C9.1: now also U3.14 (VCOM)
Other:
- moved on the sheet: R5, R6

Commit message: alt_1 V1
Parts:
- C11, C12: footprint Capacitor_THT:CP_Radial_D10.0mm_P5.00mm -> Capacitor_THT:CP_Radial_D8.0mm_P3.50mm
Changed lines of the file:
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@@
 			)
 		)
-		(property "Footprint" "Capacitor_THT:CP_Radial_D10.0mm_P5.00mm"
+		(property "Footprint" "Capacitor_THT:CP_Radial_D8.0mm_P3.50mm"
 			(at 261.3152 91.44 0)
 			(hide yes)
@@
 			)
 		)
-		(property "Footprint" "Capacitor_THT:CP_Radial_D10.0mm_P5.00mm"
+		(property "Footprint" "Capacitor_THT:CP_Radial_D8.0mm_P3.50mm"
 			(at 256.8448 91.44 0)
 			(hide yes)
